Commit message: Lower arm mounting position in URDF

File: src/mobile_platform_with_arm/resource/mobile_platform_with_arm.urdf (robot description, URDF)
Before this commit: robot mobile_platform_with_arm, 15 links, 14 joints
Joints:
- joint arm_mounting_joint: origin xyz=0.25 0 0.332 rpy=0 0 0 -> xyz=0.25 0 0.325 rpy=0 0 0
